File: Preamp socket - 1.5T 3T 7T 9.5T/Preamp socket 7T.sch (KiCad schematic (older format))
At the start: 12 parts, among them J1 In, J2 VCC, J3 Out, J4 GND, U1 Preamp

Commit message: Changed: header hole size, header to preci-dip header
Parts:
- J1, J3: footprint _Custom_footprints:PinHeader_1x03_P2.54mm_Vertical_rectangular -> _Custom:Preci-dip_PinHeader_1x03_rect
- J2: footprint Connector_PinHeader_2.54mm:PinHeader_1x02_P2.54mm_Vertical -> _Custom:Preci-dip_PinHeader_1x02_rect
- J4: footprint Connector_PinHeader_2.54mm:PinHeader_1x01_P2.54mm_Vertical -> _Custom:Preci-dip_PinHeader_1x01_rect
Changed lines of the file:
@@
 F 0 "J3" H 6672 3882 50  0000 R CNN
 F 1 "Out" H 6672 3973 50  0000 R CNN
-F 2 "_Custom_footprints:PinHeader_1x03_P2.54mm_Vertical_rectangular" H 6700 3950 50  0001 C CNN
+F 2 "_Custom:Preci-dip_PinHeader_1x03_rect" H 6700 3950 50  0001 C CNN
 F 3 "~" H 6700 3950 50  0001 C CNN
 	1    6700 3950
@@
 F 0 "J1" H 4508 4231 50  0000 C CNN
 F 1 "In" H 4508 4140 50  0000 C CNN
-F 2 "_Custom_footprints:PinHeader_1x03_P2.54mm_Vertical_rectangular" H 4400 3950 50  0001 C CNN
+F 2 "_Custom:Preci-dip_PinHeader_1x03_rect" H 4400 3950 50  0001 C CNN
 F 3 "~" H 4400 3950 50  0001 C CNN
 	1    4400 3950
@@
 F 0 "J2" V 5362 3194 50  0000 L CNN
 F 1 "VCC" V 5453 3194 50  0000 L CNN
-F 2 "Connector_PinHeader_2.54mm:PinHeader_1x02_P2.54mm_Vertical" H 5300 3150 50  0001 C CNN
+F 2 "_Custom:Preci-dip_PinHeader_1x02_rect" H 5300 3150 50  0001 C CNN
 F 3 "~" H 5300 3150 50  0001 C CNN
 	1    5300 3150
@@
 F 0 "J4" V 5454 4562 50  0000 R CNN
 F 1 "GND" V 5363 4562 50  0000 R CNN
-F 2 "Connector_PinHeader_2.54mm:PinHeader_1x01_P2.54mm_Vertical" H 5300 4650 50  0001 C CNN
+F 2 "_Custom:Preci-dip_PinHeader_1x01_rect" H 5300 4650 50  0001 C CNN
 F 3 "~" H 5300 4650 50  0001 C CNN
 	1    5300 4650
