File: Preamp socket - 1.5T 3T 7T 9.5T/Preamp socket 7T.sch (KiCad schematic (older format))
At the start: 12 parts, among them J1 In, J2 VCC, J3 Out, J4 GND, U1 Preamp

Commit message: Rescue libraries, small changes.V0.3
Parts:
- removed S1, S3: shield_clip, _Custom:S0971-46R-shield_clip, symbol _Custom:shield_clip
- added Sh1: RF_Shield_One_Piece, _Custom:Shield_15mm_20mm, symbol Device:RF_Shield_One_Piece
- G1: symbol _Custom:UMC_logo -> Preamp-socket-7T-rescue:UMC_logo-_Custom
- S2, S4, S5, S6: symbol _Custom:shield_clip -> Preamp-socket-7T-rescue:shield_clip-_Custom
- U1: footprint _Custom_footprints:Preamp_WMA7RA-R5 -> _Custom:Preamp_WMA7RA-R5; symbol _Custom:Preamp -> Preamp-socket-7T-rescue:Preamp-_Custom
Connections:
- wire segments 17 -> 14
- no-connect marks 0 -> 1
Changed lines of the file:
@@
 Sheet 1 1
 Title ""
-Date "2020-02-07"
-Rev ""
+Date "2021-11-24"
+Rev "v0.3"
 Comp ""
 Comment1 ""
@@
 $EndDescr
 $Comp
-L _Custom:UMC_logo G1
+L Preamp-socket-7T-rescue:UMC_logo-_Custom G1
 U 1 1 5E3C2881
 P 6450 7250
@@
 $EndComp
 $Comp
-L _Custom:Preamp U1
+L Preamp-socket-7T-rescue:Preamp-_Custom U1
 U 1 1 5E3C2E6D
 P 5400 3950
 F 0 "U1" H 5744 3996 50  0000 L CNN
 F 1 "Preamp" H 5744 3905 50  0000 L CNN
-F 2 "_Custom_footprints:Preamp_WMA7RA-R5" H 5750 3650 50  0001 L CNN
+F 2 "_Custom:Preamp_WMA7RA-R5" H 5750 3650 50  0001 L CNN
 F 3 "" H 5550 4100 50  0001 C CNN
 	1    5400 3950
@@
 L power:GND #PWR0101
 U 1 1 5E3C9C5B
-P 4900 4450
-F 0 "#PWR0101" H 4900 4200 50  0001 C CNN
-F 1 "GND" H 4905 4277 50  0000 C CNN
-F 2 "" H 4900 4450 50  0001 C CNN
-F 3 "" H 4900 4450 50  0001 C CNN
-	1    4900 4450
-	1    0    0    -1
-$EndComp
-Wire Wire Line
-	4900 4450 5300 4450
+P 5100 4450
+F 0 "#PWR0101" H 5100 4200 50  0001 C CNN
+F 1 "GND" H 5105 4277 50  0000 C CNN
+F 2 "" H 5100 4450 50  0001 C CNN
+F 3 "" H 5100 4450 50  0001 C CNN
+	1    5100 4450
+	1    0    0    -1
+$EndComp
+Wire Wire Line
+	5100 4450 5300 4450
 $Comp
 L power:GND #PWR0102
@@
 	5200 3350 5200 3400
 $Comp
-L _Custom:shield_clip S1
-U 1 1 5E42AE65
-P 6050 3050
-F 0 "S1" H 6000 3300 50  0000 L CNN
-F 1 "shield_clip" H 5850 3200 50  0000 L CNN
-F 2 "_Custom:S0971-46R-shield_clip" V 6000 3050 50  0001 C CNN
-F 3 "" V 6000 3050 50  0001 C CNN
-	1    6050 3050
-	1    0    0    -1
-$EndComp
-$Comp
-L _Custom:shield_clip S2
+L Preamp-socket-7T-rescue:shield_clip-_Custom S2
 U 1 1 5E42B471
-P 6500 3050
-F 0 "S2" H 6450 3300 50  0000 L CNN
-F 1 "shield_clip" H 6300 3200 50  0000 L CNN
-F 2 "_Custom:S0971-46R-shield_clip" V 6450 3050 50  0001 C CNN
-F 3 "" V 6450 3050 50  0001 C CNN
-	1    6500 3050
-	1    0    0    -1
-$EndComp
-$Comp
-L _Custom:shield_clip S3
-U 1 1 5E42B814
-P 6950 3050
-F 0 "S3" H 6900 3300 50  0000 L CNN
-F 1 "shield_clip" H 6750 3200 50  0000 L CNN
-F 2 "_Custom:S0971-46R-shield_clip" V 6900 3050 50  0001 C CNN
-F 3 "" V 6900 3050 50  0001 C CNN
-	1    6950 3050
-	1    0    0    -1
-$EndComp
-$Comp
-L _Custom:shield_clip S4
+P 6150 3100
+F 0 "S2" H 6100 3350 50  0000 L CNN
+F 1 "shield_clip" H 5950 3250 50  0000 L CNN
+F 2 "_Custom:S0971-46R-shield_clip" V 6100 3100 50  0001 C CNN
+F 3 "" V 6100 3100 50  0001 C CNN
+	1    6150 3100
+	1    0    0    -1
+$EndComp
+$Comp
+L Preamp-socket-7T-rescue:shield_clip-_Custom S4
 U 1 1 5E42BC69
-P 7400 3050
-F 0 "S4" H 7350 3300 50  0000 L CNN
-F 1 "shield_clip" H 7200 3200 50  0000 L CNN
-F 2 "_Custom:S0971-46R-shield_clip" V 7350 3050 50  0001 C CNN
-F 3 "" V 7350 3050 50  0001 C CNN
-	1    7400 3050
-	1    0    0    -1
-$EndComp
-Wire Wire Line
-	7400 3150 6950 3150
-Connection ~ 6500 3150
-Wire Wire Line
-	6500 3150 6050 3150
-Connection ~ 6950 3150
-Wire Wire Line
-	6950 3150 6700 3150
+P 6650 3100
+F 0 "S4" H 6600 3350 50  0000 L CNN
+F 1 "shield_clip" H 6450 3250 50  0000 L CNN
+F 2 "_Custom:S0971-46R-shield_clip" V 6600 3100 50  0001 C CNN
+F 3 "" V 6600 3100 50  0001 C CNN
+	1    6650 3100
+	1    0    0    -1
+$EndComp
 $Comp
 L power:GND #PWR0107
 U 1 1 5E42C2E3
-P 6700 3200
-F 0 "#PWR0107" H 6700 2950 50  0001 C CNN
-F 1 "GND" H 6705 3027 50  0000 C CNN
-F 2 "" H 6700 3200 50  0001 C CNN
-F 3 "" H 6700 3200 50  0001 C CNN
-	1    6700 3200
-	1    0    0    -1
-$EndComp
-Wire Wire Line
-	6700 3200 6700 3150
-Connection ~ 6700 3150
-Wire Wire Line
-	6700 3150 6500 3150
-$Comp
-L _Custom:shield_clip S5
+P 6850 3200
+F 0 "#PWR0107" H 6850 2950 50  0001 C CNN
+F 1 "GND" H 6855 3027 50  0000 C CNN
+F 2 "" H 6850 3200 50  0001 C CNN
+F 3 "" H 6850 3200 50  0001 C CNN
+	1    6850 3200
+	1    0    0    -1
+$EndComp
+Wire Wire Line
+	6850 3200 6650 3200
+$Comp
+L Preamp-socket-7T-rescue:shield_clip-_Custom S5
 U 1 1 5E4311CB
-P 7850 3050
-F 0 "S5" H 7800 3300 50  0000 L CNN
-F 1 "shield_clip" H 7650 3200 50  0000 L CNN
-F 2 "_Custom:S0971-46R-shield_clip" V 7800 3050 50  0001 C CNN
-F 3 "" V 7800 3050 50  0001 C CNN
-	1    7850 3050
-	1    0    0    -1
-$EndComp
-$Comp
-L _Custom:shield_clip S6
+P 7100 3100
+F 0 "S5" H 7050 3350 50  0000 L CNN
+F 1 "shield_clip" H 6900 3250 50  0000 L CNN
+F 2 "_Custom:S0971-46R-shield_clip" V 7050 3100 50  0001 C CNN
+F 3 "" V 7050 3100 50  0001 C CNN
+	1    7100 3100
+	1    0    0    -1
+$EndComp
+$Comp
+L Preamp-socket-7T-rescue:shield_clip-_Custom S6
 U 1 1 5E431539
-P 8300 3050
-F 0 "S6" H 8250 3300 50  0000 L CNN
-F 1 "shield_clip" H 8100 3200 50  0000 L CNN
-F 2 "_Custom:S0971-46R-shield_clip" V 8250 3050 50  0001 C CNN
-F 3 "" V 8250 3050 50  0001 C CNN
-	1    8300 3050
-	1    0    0    -1
-$EndComp
-Wire Wire Line
-	8300 3150 7850 3150
-Connection ~ 7400 3150
-Connection ~ 7850 3150
-Wire Wire Line
-	7850 3150 7400 3150
+P 7550 3100
+F 0 "S6" H 7500 3350 50  0000 L CNN
+F 1 "shield_clip" H 7350 3250 50  0000 L CNN
+F 2 "_Custom:S0971-46R-shield_clip" V 7500 3100 50  0001 C CNN
+F 3 "" V 7500 3100 50  0001 C CNN
+	1    7550 3100
+	1    0    0    -1
+$EndComp
+Wire Wire Line
+	7550 3200 7100 3200
+Connection ~ 6650 3200
+Connection ~ 7100 3200
+Wire Wire Line
+	7100 3200 6850 3200
+Wire Wire Line
+	6150 3200 6650 3200
+Connection ~ 6850 3200
+$Comp
+L Device:RF_Shield_One_Piece Sh1
+U 1 1 5EAADD11
+P 7600 4600
+F 0 "Sh1" H 8230 4589 50  0000 L CNN
+F 1 "RF_Shield_One_Piece" H 8230 4498 50  0000 L CNN
+F 2 "_Custom:Shield_15mm_20mm" H 7600 4500 50  0001 C CNN
+F 3 "~" H 7600 4500 50  0001 C CNN
+	1    7600 4600
+	1    0    0    -1
+$EndComp
+NoConn ~ 7600 5000
 $EndSCHEMATC
