File: Preamp socket - 1T/Preamp socket 1T.sch (KiCad schematic (older format))
At the start: 12 parts, among them J1 In, J2 VCC, J3 Out, J4 GND, U1 Preamp

Commit message: Changed: header hole size, header to preci-dip header
Parts:
- J1, J3: footprint _Custom_footprints:PinHeader_1x03_P2.54mm_Vertical_rectangular -> _Custom:Preci-dip_PinHeader_1x03_rect
- J2: footprint Connector_PinHeader_2.54mm:PinHeader_1x02_P2.54mm_Vertical -> _Custom:Preci-dip_PinHeader_1x02_rect
- J4: footprint Connector_PinHeader_2.54mm:PinHeader_1x01_P2.54mm_Vertical -> _Custom:Preci-dip_PinHeader_1x01_rect
Changed lines of the file:
@@
 F 0 "J3" H 6672 3882 50  0000 R CNN
 F 1 "Out" H 6672 3973 50  0000 R CNN
-F 2 "_Custom_footprints:PinHeader_1x03_P2.54mm_Vertical_rectangular" H 6700 3950 50  0001 C CNN
+F 2 "_Custom:Preci-dip_PinHeader_1x03_rect" H 6700 3950 50  0001 C CNN
 F 3 "~" H 6700 3950 50  0001 C CNN
 	1    6700 3950
@@
 F 0 "J1" H 4508 4231 50  0000 C CNN
 F 1 "In" H 4508 4140 50  0000 C CNN
-F 2 "_Custom_footprints:PinHeader_1x03_P2.54mm_Vertical_rectangular" H 4400 3950 50  0001 C CNN
+F 2 "_Custom:Preci-dip_PinHeader_1x03_rect" H 4400 3950 50  0001 C CNN
 F 3 "~" H 4400 3950 50  0001 C CNN
 	1    4400 3950
@@
 F 0 "J2" V 5362 3194 50  0000 L CNN
 F 1 "VCC" V 5453 3194 50  0000 L CNN
-F 2 "Connector_PinHeader_2.54mm:PinHeader_1x02_P2.54mm_Vertical" H 5300 3150 50  0001 C CNN
+F 2 "_Custom:Preci-dip_PinHeader_1x02_rect" H 5300 3150 50  0001 C CNN
 F 3 "~" H 5300 3150 50  0001 C CNN
 	1    5300 3150
@@
 F 0 "J4" V 5454 4562 50  0000 R CNN
 F 1 "GND" V 5363 4562 50  0000 R CNN
-F 2 "Connector_PinHeader_2.54mm:PinHeader_1x01_P2.54mm_Vertical" H 5300 4650 50  0001 C CNN
+F 2 "_Custom:Preci-dip_PinHeader_1x01_rect" H 5300 4650 50  0001 C CNN
 F 3 "~" H 5300 4650 50  0001 C CNN
 	1    5300 4650

Commit message: Part of previous commit..
Parts:
- removed S1, S3: shield_clip, _Custom:S0971-46R-shield_clip, symbol _Custom:shield_clip
- added Sh1: RF_Shield_One_Piece, _Custom:Shield_15mm_20mm, symbol Device:RF_Shield_One_Piece
- G1: symbol _Custom:UMC_logo -> Preamp-socket-1T-rescue:UMC_logo-_Custom
- S2, S4, S5, S6: symbol _Custom:shield_clip -> Preamp-socket-1T-rescue:shield_clip-_Custom
- U1: symbol _Custom:Preamp -> Preamp-socket-1T-rescue:Preamp-_Custom
Connections:
- wire segments 17 -> 14
- no-connect marks 0 -> 1
Changed lines of the file:
@@
 Sheet 1 1
 Title ""
-Date "2020-02-07"
-Rev ""
+Date "2021-11-24"
+Rev "v0.3"
 Comp ""
 Comment1 ""
@@
 $EndDescr
 $Comp
-L _Custom:UMC_logo G1
+L Preamp-socket-1T-rescue:UMC_logo-_Custom G1
 U 1 1 5E3C2881
 P 6450 7250
@@
 $EndComp
 $Comp
-L _Custom:Preamp U1
+L Preamp-socket-1T-rescue:Preamp-_Custom U1
 U 1 1 5E3C2E6D
 P 5400 3950
@@
 L power:GND #PWR0101
 U 1 1 5E3C9C5B
-P 4900 4450
-F 0 "#PWR0101" H 4900 4200 50  0001 C CNN
-F 1 "GND" H 4905 4277 50  0000 C CNN
-F 2 "" H 4900 4450 50  0001 C CNN
-F 3 "" H 4900 4450 50  0001 C CNN
-	1    4900 4450
-	1    0    0    -1
-$EndComp
-Wire Wire Line
-	4900 4450 5300 4450
+P 5100 4450
+F 0 "#PWR0101" H 5100 4200 50  0001 C CNN
+F 1 "GND" H 5105 4277 50  0000 C CNN
+F 2 "" H 5100 4450 50  0001 C CNN
+F 3 "" H 5100 4450 50  0001 C CNN
+	1    5100 4450
+	1    0    0    -1
+$EndComp
+Wire Wire Line
+	5100 4450 5300 4450
 $Comp
 L power:GND #PWR0102
@@
 	5200 3350 5200 3400
 $Comp
-L _Custom:shield_clip S1
-U 1 1 5E42AE65
-P 6050 3050
-F 0 "S1" H 6000 3300 50  0000 L CNN
-F 1 "shield_clip" H 5850 3200 50  0000 L CNN
-F 2 "_Custom:S0971-46R-shield_clip" V 6000 3050 50  0001 C CNN
-F 3 "" V 6000 3050 50  0001 C CNN
-	1    6050 3050
-	1    0    0    -1
-$EndComp
-$Comp
-L _Custom:shield_clip S2
+L Preamp-socket-1T-rescue:shield_clip-_Custom S2
 U 1 1 5E42B471
-P 6500 3050
-F 0 "S2" H 6450 3300 50  0000 L CNN
-F 1 "shield_clip" H 6300 3200 50  0000 L CNN
-F 2 "_Custom:S0971-46R-shield_clip" V 6450 3050 50  0001 C CNN
-F 3 "" V 6450 3050 50  0001 C CNN
-	1    6500 3050
-	1    0    0    -1
-$EndComp
-$Comp
-L _Custom:shield_clip S3
-U 1 1 5E42B814
-P 6950 3050
-F 0 "S3" H 6900 3300 50  0000 L CNN
-F 1 "shield_clip" H 6750 3200 50  0000 L CNN
-F 2 "_Custom:S0971-46R-shield_clip" V 6900 3050 50  0001 C CNN
-F 3 "" V 6900 3050 50  0001 C CNN
-	1    6950 3050
-	1    0    0    -1
-$EndComp
-$Comp
-L _Custom:shield_clip S4
+P 6900 3050
+F 0 "S2" H 6850 3300 50  0000 L CNN
+F 1 "shield_clip" H 6700 3200 50  0000 L CNN
+F 2 "_Custom:S0971-46R-shield_clip" V 6850 3050 50  0001 C CNN
+F 3 "" V 6850 3050 50  0001 C CNN
+	1    6900 3050
+	1    0    0    -1
+$EndComp
+$Comp
+L Preamp-socket-1T-rescue:shield_clip-_Custom S4
 U 1 1 5E42BC69
 P 7400 3050
@@
 	1    0    0    -1
 $EndComp
-Wire Wire Line
-	7400 3150 6950 3150
-Connection ~ 6500 3150
-Wire Wire Line
-	6500 3150 6050 3150
-Connection ~ 6950 3150
-Wire Wire Line
-	6950 3150 6700 3150
 $Comp
 L power:GND #PWR0107
 U 1 1 5E42C2E3
-P 6700 3200
-F 0 "#PWR0107" H 6700 2950 50  0001 C CNN
-F 1 "GND" H 6705 3027 50  0000 C CNN
-F 2 "" H 6700 3200 50  0001 C CNN
-F 3 "" H 6700 3200 50  0001 C CNN
-	1    6700 3200
-	1    0    0    -1
-$EndComp
-Wire Wire Line
-	6700 3200 6700 3150
-Connection ~ 6700 3150
-Wire Wire Line
-	6700 3150 6500 3150
-$Comp
-L _Custom:shield_clip S5
+P 7600 3150
+F 0 "#PWR0107" H 7600 2900 50  0001 C CNN
+F 1 "GND" H 7605 2977 50  0000 C CNN
+F 2 "" H 7600 3150 50  0001 C CNN
+F 3 "" H 7600 3150 50  0001 C CNN
+	1    7600 3150
+	1    0    0    -1
+$EndComp
+Wire Wire Line
+	7600 3150 7400 3150
+$Comp
+L Preamp-socket-1T-rescue:shield_clip-_Custom S5
 U 1 1 5E4311CB
 P 7850 3050
@@
 $EndComp
 $Comp
-L _Custom:shield_clip S6
+L Preamp-socket-1T-rescue:shield_clip-_Custom S6
 U 1 1 5E431539
 P 8300 3050
@@
 Connection ~ 7850 3150
 Wire Wire Line
-	7850 3150 7400 3150
+	7850 3150 7600 3150
+Wire Wire Line
+	6900 3150 7400 3150
+Connection ~ 7600 3150
+$Comp
+L Device:RF_Shield_One_Piece Sh1
+U 1 1 5EAB1F76
+P 7850 4600
+F 0 "Sh1" H 8480 4589 50  0000 L CNN
+F 1 "RF_Shield_One_Piece" H 8480 4498 50  0000 L CNN
+F 2 "_Custom:Shield_15mm_20mm" H 7850 4500 50  0001 C CNN
+F 3 "~" H 7850 4500 50  0001 C CNN
+	1    7850 4600
+	1    0    0    -1
+$EndComp
+NoConn ~ 7850 5000
 $EndSCHEMATC
