File: Preamp socket - 1T/Preamp socket 1T.kicad_pcb (KiCad board)
At the start: 2 copper layers, 23 x 17.8 mm, 13 parts, among them J1 In, J2 VCC, J3 Out, J4 GND, U1 Preamp

Commit message: Part of previous commit..
Parts:
- removed REF**: Shield_15mm_20mm, _Custom:Shield_15mm_20mm
- removed S1, S3: shield_clip, _Custom:S0971-46R-shield_clip
- added Sh1: RF_Shield_One_Piece, _Custom:Shield_15mm_20mm, F.Cu at (157.0, 99.1)
- moved S5 0.57 mm to (163.4, 106.6)
- moved J4 0.53 mm to (156.8, 93.0)
- moved J2 0.48 mm to (156.8, 105.2)
- moved J3 0.43 mm to (165.6, 96.6)
- moved J1 0.43 mm to (148.4, 96.6)
- moved G1 0.20 mm to (164.0, 93.1)
- moved S2 0.09 mm to (151.2, 91.6)
- moved S4 0.09 mm to (151.2, 106.6)
- moved S6 0.09 mm to (162.9, 91.6)
Routing:
- net GND: track 2.50 -> 3.91 mm
Other:
- board text added: "04/2020 v0.3"
- board text removed: "03/2020 v0.2"
- board text removed: "DW"

Commit message: Correct board thickness and solder mask clearance
Other:
- rule pad_to_mask_clearance: 0.051 -> 0
Changed lines of the file:
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@@
     (pad_size 1.7 1.7)
     (pad_drill 1.45)
-    (pad_to_mask_clearance 0.051)
-    (solder_mask_min_width 0.25)
+    (pad_to_mask_clearance 0)
     (aux_axis_origin 0 0)
     (grid_origin 157.0228 99.1108)

Commit message: Updated to v1.0
Other:
- board text added: "04/2020 v1.0"
- board text removed: "04/2020 v0.3"

Commit message: Updated version date
Other:
- board text added: "11/2021 v1.0"
- board text removed: "04/2020 v1.0"
